File: Venta LW Controller.sch (KiCad schematic (older format))
At the start: 24 parts, among them J1 Conn_01x04, J2 Conn_02x05_Odd_Even, Q1 BSS138, Q2 BSS138, SW1 RST, SW2 FLASH, U1 LM2674N-3.3, U2 ESP-12F

Commit message: updated package
Parts:
- U1: footprint Package_DIP:DIP-8_W7.62mm_SMDSocket_SmallPads -> Package_SO:SOIC-8_3.9x4.9mm_P1.27mm
Other:
- moved on the sheet: C3, L1
Changed lines of the file:
@@
 F 0 "U1" H 2600 1767 50  0000 C CNN
 F 1 "LM2674N-3.3" H 2600 1676 50  0000 C CNN
-F 2 "Package_DIP:DIP-8_W7.62mm_SMDSocket_SmallPads" H 2650 950 50  0001 L CIN
+F 2 "Package_SO:SOIC-8_3.9x4.9mm_P1.27mm" H 2650 950 50  0001 L CIN
 F 3 "http://www.ti.com/lit/ds/symlink/lm2674.pdf" H 2600 1300 50  0001 C CNN
 F 4 "TME" H 2600 1300 50  0001 C CNN "Supplier"
@@
 Wire Wire Line
 	3250 1850 2600 1850
+$Comp
+L Device:L_Small L1
+U 1 1 5D7A40F0
+P 4100 1500
+F 0 "L1" V 4285 1500 50  0000 C CNN
+F 1 "100u" V 4194 1500 50  0000 C CNN
+F 2 "Inductor_SMD:L_12x12mm_H8mm" H 4100 1500 50  0001 C CNN
+F 3 "~" H 4100 1500 50  0001 C CNN
+F 4 "TME" H 4100 1500 50  0001 C CNN "Supplier"
+F 5 "DE1207-120" H 4100 1500 50  0001 C CNN "Supplier Part"
+	1    4100 1500
+	0    -1   -1   0
+$EndComp
 Wire Wire Line
 	3250 1500 3550 1500
@@
 	3550 1300 3550 1500
 Connection ~ 3550 1500
-Wire Wire Line
-	4100 1850 3250 1850
+$Comp
+L Device:CP_Small C3
+U 1 1 5D7A5ACA
+P 4300 1700
+F 0 "C3" H 4388 1746 50  0000 L CNN
+F 1 "100u" H 4388 1655 50  0000 L CNN
+F 2 "Capacitor_Tantalum_SMD:CP_EIA-6032-28_Kemet-C" H 4300 1700 50  0001 C CNN
+F 3 "~" H 4300 1700 50  0001 C CNN
+F 4 "TME" H 4300 1700 50  0001 C CNN "Supplier"
+F 5 "TPSC107M010R0100" H 4300 1700 50  0001 C CNN "Supplier Part"
+	1    4300 1700
+	1    0    0    -1
+$EndComp
+Wire Wire Line
+	4300 1800 4300 1850
+Wire Wire Line
+	4300 1850 3250 1850
 Connection ~ 3250 1850
 Wire Wire Line
+	4200 1500 4300 1500
+Wire Wire Line
 	3100 1100 3150 1100
 Wire Wire Line
 	3150 1100 3150 950
-Wire Wire Line
-	3150 950  4100 950
 Text GLabel 1150 4900 0    50   Input ~ 0
 +3.3V
@@
 GPIO14
 Wire Wire Line
-	3950 1500 4100 1500
-$Comp
-L Device:L_Small L1
-U 1 1 5D7A40F0
-P 3850 1500
-F 0 "L1" V 4035 1500 50  0000 C CNN
-F 1 "100u" V 3944 1500 50  0000 C CNN
-F 2 "Inductor_SMD:L_12x12mm_H8mm" H 3850 1500 50  0001 C CNN
-F 3 "~" H 3850 1500 50  0001 C CNN
-F 4 "TME" H 3850 1500 50  0001 C CNN "Supplier"
-F 5 "DE1207-120" H 3850 1500 50  0001 C CNN "Supplier Part"
-	1    3850 1500
-	0    -1   -1   0
-$EndComp
-Wire Wire Line
-	4100 1750 4100 1850
-$Comp
-L Device:CP_Small C3
-U 1 1 5D7A5ACA
-P 4100 1650
-F 0 "C3" H 4188 1696 50  0000 L CNN
-F 1 "100u" H 4188 1605 50  0000 L CNN
-F 2 "Capacitor_Tantalum_SMD:CP_EIA-6032-28_Kemet-C" H 4100 1650 50  0001 C CNN
-F 3 "~" H 4100 1650 50  0001 C CNN
-F 4 "TME" H 4100 1650 50  0001 C CNN "Supplier"
-F 5 "TPSC107M010R0100" H 4100 1650 50  0001 C CNN "Supplier Part"
-	1    4100 1650
-	1    0    0    -1
-$EndComp
-Wire Wire Line
-	3550 1500 3750 1500
-Wire Wire Line
-	4100 950  4100 1500
-Connection ~ 4100 1500
-Wire Wire Line
-	4100 1500 4400 1500
-Wire Wire Line
-	4100 1550 4100 1500
+	3550 1500 4000 1500
+Wire Wire Line
+	4300 1600 4300 1500
+Connection ~ 4300 1500
+Wire Wire Line
+	4300 1500 4400 1500
+Wire Wire Line
+	4300 950  4300 1500
+Wire Wire Line
+	3150 950  4300 950
 $EndSCHEMATC
