File: Venta LW Controller.sch (KiCad schematic (older format))
At the start: 24 parts, among them J1 Conn_01x04, J2 Conn_02x05_Odd_Even, Q1 BSS138, Q2 BSS138, SW1 RST, SW2 FLASH, U1 LM2674N-3.3, U2 ESP-12F

Commit message: use usable GPIOs
Parts:
- C1: value 25u -> 22u; Supplier (none) -> TME; Supplier Part (none) -> TPSA226K010R0900
- C2: Supplier (none) -> TME; Supplier Part (none) -> 06035A100JAT2A
- C3: Supplier (none) -> TME; Supplier Part (none) -> TPSC107M010R0100
- C4: Supplier (none) -> TME; Supplier Part (none) -> CL03B103KP3NNNC
- C5: value 100u -> 47u; Supplier (none) -> TM; Supplier Part (none) -> CL21A476MQYNNNG
- C7: Supplier (none) -> TME; Supplier Part (none) -> CL10B104KO8NNNC
- D1: Supplier (none) -> TME; Supplier Part (none) -> B130-13-F
- J1: Supplier (none) -> TME; Supplier Part (none) -> ZL201-04G
- J2: Supplier (none) -> TME; Supplier Part (none) -> T821-1-10-S1
- L1: Supplier (none) -> TME; Supplier Part (none) -> DE1207-120
- Q1, Q2: Supplier (none) -> TME; Supplier Part (none) -> BSS138LT1G
- R1, R2, R3, R4, R5, R6, R7, R8: Supplier (none) -> TME; Supplier Part (none) -> SMD0603-10K-1%
- SW1, SW2: Supplier (none) -> TME; Supplier Part (none) -> TACT-67N-F
- U1: Supplier (none) -> TME; Supplier Part (none) -> LM2674M-3.3/NOP
Connections:
- net labels added: GPIO1, GPIO12, GPIO13, GPIO14, GPIO3
- net labels removed: GPIO10, GPIO6, GPIO7, GPIO8, GPIO9
- wire segments 102 -> 103
- no-connect marks 8 -> 10
Changed lines of the file:
@@
 EESchema Schematic File Version 4
-LIBS:Venta LW45-cache
+LIBS:Venta LW Controller-cache
 EELAYER 30 0
 EELAYER END
@@
 F 2 "Package_DIP:DIP-8_W7.62mm_SMDSocket_SmallPads" H 2650 950 50  0001 L CIN
 F 3 "http://www.ti.com/lit/ds/symlink/lm2674.pdf" H 2600 1300 50  0001 C CNN
+F 4 "TME" H 2600 1300 50  0001 C CNN "Supplier"
+F 5 "LM2674M-3.3/NOP" H 2600 1300 50  0001 C CNN "Supplier Part"
 	1    2600 1300
 	1    0    0    -1
@@
 P 1750 1650
 F 0 "C1" H 1838 1696 50  0000 L CNN
-F 1 "25u" H 1838 1605 50  0000 L CNN
+F 1 "22u" H 1838 1605 50  0000 L CNN
 F 2 "Capacitor_Tantalum_SMD:CP_EIA-3216-18_Kemet-A" H 1750 1650 50  0001 C CNN
 F 3 "~" H 1750 1650 50  0001 C CNN
+F 4 "TME" H 1750 1650 50  0001 C CNN "Supplier"
+F 5 "TPSA226K010R0900" H 1750 1650 50  0001 C CNN "Supplier Part"
 	1    1750 1650
 	1    0    0    -1
@@
 F 2 "Capacitor_SMD:C_0603_1608Metric" H 3350 1300 50  0001 C CNN
 F 3 "~" H 3350 1300 50  0001 C CNN
+F 4 "TME" H 3350 1300 50  0001 C CNN "Supplier"
+F 5 "06035A100JAT2A" H 3350 1300 50  0001 C CNN "Supplier Part"
 	1    3350 1300
 	0    -1   -1   0
@@
 F 2 "Diode_SMD:D_SMA" V 3250 1650 50  0001 C CNN
 F 3 "~" V 3250 1650 50  0001 C CNN
+F 4 "TME" H 3250 1650 50  0001 C CNN "Supplier"
+F 5 "B130-13-F" H 3250 1650 50  0001 C CNN "Supplier Part"
 	1    3250 1650
 	0    1    1    0
@@
 F 2 "Inductor_SMD:L_12x12mm_H8mm" H 4100 1500 50  0001 C CNN
 F 3 "~" H 4100 1500 50  0001 C CNN
+F 4 "TME" H 4100 1500 50  0001 C CNN "Supplier"
+F 5 "DE1207-120" H 4100 1500 50  0001 C CNN "Supplier Part"
 	1    4100 1500
 	0    -1   -1   0
@@
 F 2 "Capacitor_Tantalum_SMD:CP_EIA-6032-28_Kemet-C" H 3850 1650 50  0001 C CNN
 F 3 "~" H 3850 1650 50  0001 C CNN
+F 4 "TME" H 3850 1650 50  0001 C CNN "Supplier"
+F 5 "TPSC107M010R0100" H 3850 1650 50  0001 C CNN "Supplier Part"
 	1    3850 1650
 	1    0    0    -1
@@
 F 2 "Capacitor_SMD:C_0805_2012Metric" H 1600 5150 50  0001 C CNN
 F 3 "~" H 1600 5150 50  0001 C CNN
+F 4 "TME" H 1600 5150 50  0001 C CNN "Supplier"
+F 5 "CL03B103KP3NNNC" H 1600 5150 50  0001 C CNN "Supplier Part"
 	1    1600 5150
 	1    0    0    -1
@@
 P 2000 5150
 F 0 "C5" H 2092 5196 50  0000 L CNN
-F 1 "100u" H 2092 5105 50  0000 L CNN
+F 1 "47u" H 2092 5105 50  0000 L CNN
 F 2 "Capacitor_SMD:C_0805_2012Metric" H 2000 5150 50  0001 C CNN
 F 3 "~" H 2000 5150 50  0001 C CNN
+F 4 "TM" H 2000 5150 50  0001 C CNN "Supplier"
+F 5 "CL21A476MQYNNNG" H 2000 5150 50  0001 C CNN "Supplier Part"
 	1    2000 5150
 	1    0    0    -1
@@
 F 2 "Resistor_SMD:R_0603_1608Metric" H 1850 3900 50  0001 C CNN
 F 3 "~" H 1850 3900 50  0001 C CNN
+F 4 "TME" H 1850 3900 50  0001 C CNN "Supplier"
+F 5 "SMD0603-10K-1%" H 1850 3900 50  0001 C CNN "Supplier Part"
 	1    1850 3900
 	0    -1   -1   0
@@
 F 2 "Resistor_SMD:R_0603_1608Metric" H 1850 3450 50  0001 C CNN
 F 3 "~" H 1850 3450 50  0001 C CNN
+F 4 "TME" H 1850 3450 50  0001 C CNN "Supplier"
+F 5 "SMD0603-10K-1%" H 1850 3450 50  0001 C CNN "Supplier Part"
 	1    1850 3450
 	0    -1   -1   0
@@
 F 2 "Resistor_SMD:R_0603_1608Metric" H 4950 4600 50  0001 C CNN
 F 3 "~" H 4950 4600 50  0001 C CNN
+F 4 "TME" H 4950 4600 50  0001 C CNN "Supplier"
+F 5 "SMD0603-10K-1%" H 4950 4600 50  0001 C CNN "Supplier Part"
 	1    4950 4600
 	-1   0    0    1
@@
 Wire Wire Line
 	4950 4900 4950 5100
-Text GLabel 4850 3700 2    50   Output ~ 0
+Text GLabel 5350 3700 2    50   Output ~ 0
 TXD
-Text GLabel 4850 3800 2    50   Input ~ 0
+Text GLabel 5350 3800 2    50   Input ~ 0
 RXD
-Wire Wire Line
-	4650 3700 4850 3700
-Wire Wire Line
-	4650 3800 4850 3800
 NoConn ~ 2850 4000
 NoConn ~ 4650 4200
@@
 F 2 "Package_TO_SOT_SMD:SOT-23" H 7400 2900 50  0001 C CNN
 F 3 "~" H 7200 2800 50  0001 C CNN
+F 4 "TME" H 7200 2800 50  0001 C CNN "Supplier"
+F 5 "BSS138LT1G" H 7200 2800 50  0001 C CNN "Supplier Part"
 	1    7200 2800
 	1    0    0    -1
@@
 F 2 "Package_TO_SOT_SMD:SOT-23" H 9300 2900 50  0001 C CNN
 F 3 "~" H 9100 2800 50  0001 C CNN
+F 4 "TME" H 9100 2800 50  0001 C CNN "Supplier"
+F 5 "BSS138LT1G" H 9100 2800 50  0001 C CNN "Supplier Part"
 	1    9100 2800
 	1    0    0    -1
@@
 F 2 "Resistor_SMD:R_0603_1608Metric" H 7900 5400 50  0001 C CNN
 F 3 "~" H 7900 5400 50  0001 C CNN
+F 4 "TME" H 7900 5400 50  0001 C CNN "Supplier"
+F 5 "SMD0603-10K-1%" H 7900 5400 50  0001 C CNN "Supplier Part"
 	1    7900 5400
 	0    1    1    0
@@
 LED_POWER
 Text GLabel 8350 5400 2    50   Output ~ 0
-GPIO6
+GPIO3
 Wire Wire Line
 	7450 5400 7800 5400
@@
 F 2 "Resistor_SMD:R_0603_1608Metric" H 7900 4000 50  0001 C CNN
 F 3 "~" H 7900 4000 50  0001 C CNN
+F 4 "TME" H 7900 4000 50  0001 C CNN "Supplier"
+F 5 "SMD0603-10K-1%" H 7900 4000 50  0001 C CNN "Supplier Part"
 	1    7900 4000
 	0    1    1    0
@@
 LED_LOW
 Text GLabel 8350 4000 2    50   Output ~ 0
-GPIO7
+GPIO13
 Wire Wire Line
 	7450 4000 7800 4000
@@
 F 2 "Resistor_SMD:R_0603_1608Metric" H 7900 5050 50  0001 C CNN
 F 3 "~" H 7900 5050 50  0001 C CNN
+F 4 "TME" H 7900 5050 50  0001 C CNN "Supplier"
+F 5 "SMD0603-10K-1%" H 7900 5050 50  0001 C CNN "Supplier Part"
 	1    7900 5050
 	0    1    1    0
@@
 LED_MID
 Text GLabel 8350 5050 2    50   Output ~ 0
-GPIO8
+GPIO1
 Wire Wire Line
 	7450 5050 7800 5050
@@
 F 2 "Resistor_SMD:R_0603_1608Metric" H 7900 4350 50  0001 C CNN
 F 3 "~" H 7900 4350 50  0001 C CNN
+F 4 "TME" H 7900 4350 50  0001 C CNN "Supplier"
+F 5 "SMD0603-10K-1%" H 7900 4350 50  0001 C CNN "Supplier Part"
 	1    7900 4350
 	0    1    1    0
@@
 LED_HIGH
 Text GLabel 8350 4350 2    50   Output ~ 0
-GPIO9
+GPIO12
 Wire Wire Line
 	7450 4350 7800 4350
@@
 F 2 "Resistor_SMD:R_0603_1608Metric" H 7900 4700 50  0001 C CNN
 F 3 "~" H 7900 4700 50  0001 C CNN
+F 4 "TME" H 7900 4700 50  0001 C CNN "Supplier"
+F 5 "SMD0603-10K-1%" H 7900 4700 50  0001 C CNN "Supplier Part"
 	1    7900 4700
 	0    1    1    0
@@
 LED_ERROR
 Text GLabel 8350 4700 2    50   Output ~ 0
-GPIO10
+GPIO14
 Wire Wire Line
 	7450 4700 7800 4700
 Wire Wire Line
 	8000 4700 8350 4700
-Text GLabel 4000 5100 3    50   Input ~ 0
-GPIO6
-Text GLabel 3600 5100 3    50   Input ~ 0
-GPIO7
-Text GLabel 3900 5100 3    50   Input ~ 0
-GPIO8
-Text GLabel 3700 5100 3    50   Input ~ 0
-GPIO9
-Text GLabel 3800 5100 3    50   Input ~ 0
-GPIO10
-Wire Wire Line
-	3600 5100 3600 4900
-Wire Wire Line
-	3700 4900 3700 5100
-Wire Wire Line
-	3800 4900 3800 5100
-Wire Wire Line
-	3900 4900 3900 5100
-Wire Wire Line
-	4000 4900 4000 5100
-NoConn ~ 2850 4300
-NoConn ~ 2850 4200
 NoConn ~ 2850 3800
 NoConn ~ 3500 4900
-NoConn ~ 2850 4100
 Text GLabel 4850 4100 2    50   Output ~ 0
 FLASH
@@
 F 2 "Capacitor_SMD:C_0805_2012Metric" H 2450 3200 50  0001 C CNN
 F 3 "~" H 2450 3200 50  0001 C CNN
+F 4 "TME" H 2450 3200 50  0001 C CNN "Supplier"
+F 5 "CL10B104KO8NNNC" H 2450 3200 50  0001 C CNN "Supplier Part"
 	1    2450 3200
 	1    0    0    -1
@@
 F 2 "Button_Switch_THT:SW_PUSH_6mm_H5mm" H 1700 6400 50  0001 C CNN
 F 3 "~" H 1700 6400 50  0001 C CNN
+F 4 "TME" H 1700 6400 50  0001 C CNN "Supplier"
+F 5 "TACT-67N-F" H 1700 6400 50  0001 C CNN "Supplier Part"
 	1    1700 6400
 	1    0    0    -1
@@
 F 2 "Button_Switch_THT:SW_PUSH_6mm_H5mm" H 1700 7050 50  0001 C CNN
 F 3 "~" H 1700 7050 50  0001 C CNN
+F 4 "TME" H 1700 7050 50  0001 C CNN "Supplier"
+F 5 "TACT-67N-F" H 1700 7050 50  0001 C CNN "Supplier Part"
 	1    1700 7050
 	1    0    0    -1
@@
 F 2 "Connector_PinHeader_2.54mm:PinHeader_1x04_P2.54mm_Vertical" H 3750 6800 50  0001 C CNN
 F 3 "~" H 3750 6800 50  0001 C CNN
+F 4 "TME" H 3750 6800 50  0001 C CNN "Supplier"
+F 5 "ZL201-04G" H 3750 6800 50  0001 C CNN "Supplier Part"
 	1    3750 6800
 	1    0    0    -1
@@
 F 2 "Connector_IDC:IDC-Header_2x05_P2.54mm_Vertical" H 8350 1350 50  0001 C CNN
 F 3 "~" H 8350 1350 50  0001 C CNN
+F 4 "TME" H 8350 1350 50  0001 C CNN "Supplier"
+F 5 "T821-1-10-S1" H 8350 1350 50  0001 C CNN "Supplier Part"
 	1    8350 1350
 	1    0    0    -1
 $EndComp
+Text GLabel 5350 3900 2    50   Input ~ 0
+GPIO3
+Text GLabel 5350 3600 2    50   Input ~ 0
+GPIO1
+Wire Wire Line
+	4650 3800 5250 3800
+Wire Wire Line
+	5250 3800 5250 3900
+Wire Wire Line
+	5250 3900 5350 3900
+Connection ~ 5250 3800
+Wire Wire Line
+	5250 3800 5350 3800
+Wire Wire Line
+	4650 3700 5250 3700
+Wire Wire Line
+	5250 3700 5250 3600
+Wire Wire Line
+	5250 3600 5350 3600
+Connection ~ 5250 3700
+Wire Wire Line
+	5250 3700 5350 3700
+NoConn ~ 3600 4900
+NoConn ~ 3700 4900
+NoConn ~ 3800 4900
+NoConn ~ 3900 4900
+NoConn ~ 4000 4900
+Text GLabel 2850 4300 0    50   Input ~ 0
+GPIO13
+Text GLabel 2850 4200 0    50   Input ~ 0
+GPIO12
+Text GLabel 2850 4100 0    50   Input ~ 0
+GPIO14
 $EndSCHEMATC

Commit message: switched to ESP32
Parts:
- removed C7: 100n, Capacitor_SMD:C_0805_2012Metric, symbol Device:C_Small
- removed R1, R3: 10k, Resistor_SMD:R_0603_1608Metric, symbol Device:R_Small
- removed U2: ESP-12F, ALITECS:ESP-12E, symbol ALITECS:ESP-12F
- added U2: ESP32-WROOM-32, RF_Module:ESP32-WROOM-32, symbol RF_Module:ESP32-WROOM-32
Connections:
- net labels added: GPIO16, GPIO17, GPIO18, GPIO19, GPIO21, GPIO22, GPIO23
- net labels removed: GPIO1, GPIO12, GPIO13, GPIO14, GPIO3, GPIO4, GPIO5
- wire segments 103 -> 90
- no-connect marks 10 -> 1
Other:
- moved on the sheet: C4, C5, R2

Commit message: corrected circuit and updated layout
Connections:
- net +3.3V: now also C3.1, U1.4 (FB)
- net at C2.2, D1.1 (K), L1.1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: no longer C3.1, U1.4 (FB)
Other:
- moved on the sheet: C3, L1
Changed lines of the file:
@@
 Wire Wire Line
 	2600 1850 2600 1700
-Text GLabel 4400 1500 2    50   Output ~ 0
+Text GLabel 4300 1500 2    50   Output ~ 0
 +3.3V
 Wire Wire Line
@@
 L Device:L_Small L1
 U 1 1 5D7A40F0
-P 4100 1500
-F 0 "L1" V 4285 1500 50  0000 C CNN
-F 1 "100u" V 4194 1500 50  0000 C CNN
-F 2 "Inductor_SMD:L_12x12mm_H8mm" H 4100 1500 50  0001 C CNN
-F 3 "~" H 4100 1500 50  0001 C CNN
-F 4 "TME" H 4100 1500 50  0001 C CNN "Supplier"
-F 5 "DE1207-120" H 4100 1500 50  0001 C CNN "Supplier Part"
-	1    4100 1500
+P 3800 1500
+F 0 "L1" V 3985 1500 50  0000 C CNN
+F 1 "100u" V 3894 1500 50  0000 C CNN
+F 2 "Inductor_SMD:L_12x12mm_H8mm" H 3800 1500 50  0001 C CNN
+F 3 "~" H 3800 1500 50  0001 C CNN
+F 4 "TME" H 3800 1500 50  0001 C CNN "Supplier"
+F 5 "DE1207-120" H 3800 1500 50  0001 C CNN "Supplier Part"
+	1    3800 1500
 	0    -1   -1   0
 $EndComp
-Wire Wire Line
-	3250 1500 3550 1500
 Connection ~ 3250 1500
 Wire Wire Line
@@
 	3550 1300 3550 1500
 Connection ~ 3550 1500
-Wire Wire Line
-	3550 1500 3850 1500
 $Comp
 L Device:CP_Small C3
 U 1 1 5D7A5ACA
-P 3850 1650
-F 0 "C3" H 3938 1696 50  0000 L CNN
-F 1 "100u" H 3938 1605 50  0000 L CNN
-F 2 "Capacitor_Tantalum_SMD:CP_EIA-6032-28_Kemet-C" H 3850 1650 50  0001 C CNN
-F 3 "~" H 3850 1650 50  0001 C CNN
-F 4 "TME" H 3850 1650 50  0001 C CNN "Supplier"
-F 5 "TPSC107M010R0100" H 3850 1650 50  0001 C CNN "Supplier Part"
-	1    3850 1650
-	1    0    0    -1
-$EndComp
-Wire Wire Line
-	3850 1550 3850 1500
-Connection ~ 3850 1500
-Wire Wire Line
-	3850 1500 4000 1500
-Wire Wire Line
-	3850 1750 3850 1850
-Wire Wire Line
-	3850 1850 3250 1850
+P 4000 1650
+F 0 "C3" H 4088 1696 50  0000 L CNN
+F 1 "100u" H 4088 1605 50  0000 L CNN
+F 2 "Capacitor_Tantalum_SMD:CP_EIA-6032-28_Kemet-C" H 4000 1650 50  0001 C CNN
+F 3 "~" H 4000 1650 50  0001 C CNN
+F 4 "TME" H 4000 1650 50  0001 C CNN "Supplier"
+F 5 "TPSC107M010R0100" H 4000 1650 50  0001 C CNN "Supplier Part"
+	1    4000 1650
+	1    0    0    -1
+$EndComp
+Wire Wire Line
+	4000 1750 4000 1850
+Wire Wire Line
+	4000 1850 3250 1850
 Connection ~ 3250 1850
 Wire Wire Line
-	4200 1500 4400 1500
+	3900 1500 4000 1500
 Wire Wire Line
 	3100 1100 3150 1100
@@
 	3150 1100 3150 950
 Wire Wire Line
-	3150 950  3850 950
-Wire Wire Line
-	3850 950  3850 1500
+	3150 950  4000 950
+Wire Wire Line
+	4000 950  4000 1500
 Text GLabel 2150 2300 0    50   Input ~ 0
 +3.3V
@@
 Wire Wire Line
 	4350 3200 4450 3200
+Connection ~ 4000 1500
+Wire Wire Line
+	4000 1500 4300 1500
+Wire Wire Line
+	3250 1500 3550 1500
+Wire Wire Line
+	4000 1550 4000 1500
+Wire Wire Line
+	3550 1500 3700 1500
 $EndSCHEMATC

Commit message: updated package
Parts:
- U1: footprint Package_DIP:DIP-8_W7.62mm_SMDSocket_SmallPads -> Package_SO:SOIC-8_3.9x4.9mm_P1.27mm
Changed lines of the file:
@@
 F 0 "U1" H 2600 1767 50  0000 C CNN
 F 1 "LM2674N-3.3" H 2600 1676 50  0000 C CNN
-F 2 "Package_DIP:DIP-8_W7.62mm_SMDSocket_SmallPads" H 2650 950 50  0001 L CIN
+F 2 "Package_SO:SOIC-8_3.9x4.9mm_P1.27mm" H 2650 950 50  0001 L CIN
 F 3 "http://www.ti.com/lit/ds/symlink/lm2674.pdf" H 2600 1300 50  0001 C CNN
 F 4 "TME" H 2600 1300 50  0001 C CNN "Supplier"

Commit message: updated values
Parts:
- C1: value 22u -> 22uF
- C2: value 0.01u -> 0.01uF
- C3: value 100u -> 100uF
- C4: value 10n -> 10nF
- C5: value 47u -> 47uF
- L1: value 100u -> 100uH
- R2, R4, R5, R6, R7, R8: value 10k -> 10K
Changed lines of the file:
@@
 P 1750 1650
 F 0 "C1" H 1838 1696 50  0000 L CNN
-F 1 "22u" H 1838 1605 50  0000 L CNN
+F 1 "22uF" H 1838 1605 50  0000 L CNN
 F 2 "Capacitor_Tantalum_SMD:CP_EIA-3216-18_Kemet-A" H 1750 1650 50  0001 C CNN
 F 3 "~" H 1750 1650 50  0001 C CNN
@@
 P 3350 1300
 F 0 "C2" V 3579 1300 50  0000 C CNN
-F 1 "0.01u" V 3488 1300 50  0000 C CNN
+F 1 "0.01uF" V 3488 1300 50  0000 C CNN
 F 2 "Capacitor_SMD:C_0603_1608Metric" H 3350 1300 50  0001 C CNN
 F 3 "~" H 3350 1300 50  0001 C CNN
@@
 P 3800 1500
 F 0 "L1" V 3985 1500 50  0000 C CNN
-F 1 "100u" V 3894 1500 50  0000 C CNN
+F 1 "100uH" V 3894 1500 50  0000 C CNN
 F 2 "Inductor_SMD:L_12x12mm_H8mm" H 3800 1500 50  0001 C CNN
 F 3 "~" H 3800 1500 50  0001 C CNN
@@
 P 4000 1650
 F 0 "C3" H 4088 1696 50  0000 L CNN
-F 1 "100u" H 4088 1605 50  0000 L CNN
+F 1 "100uF" H 4088 1605 50  0000 L CNN
 F 2 "Capacitor_Tantalum_SMD:CP_EIA-6032-28_Kemet-C" H 4000 1650 50  0001 C CNN
 F 3 "~" H 4000 1650 50  0001 C CNN
@@
 P 2600 2550
 F 0 "C4" H 2692 2596 50  0000 L CNN
-F 1 "10n" H 2692 2505 50  0000 L CNN
+F 1 "10nF" H 2692 2505 50  0000 L CNN
 F 2 "Capacitor_SMD:C_0805_2012Metric" H 2600 2550 50  0001 C CNN
 F 3 "~" H 2600 2550 50  0001 C CNN
@@
 P 3000 2550
 F 0 "C5" H 3092 2596 50  0000 L CNN
-F 1 "47u" H 3092 2505 50  0000 L CNN
+F 1 "47uF" H 3092 2505 50  0000 L CNN
 F 2 "Capacitor_SMD:C_0805_2012Metric" H 3000 2550 50  0001 C CNN
 F 3 "~" H 3000 2550 50  0001 C CNN
@@
 P 1850 4400
 F 0 "R2" V 2046 4400 50  0000 C CNN
-F 1 "10k" V 1955 4400 50  0000 C CNN
+F 1 "10K" V 1955 4400 50  0000 C CNN
 F 2 "Resistor_SMD:R_0603_1608Metric" H 1850 4400 50  0001 C CNN
 F 3 "~" H 1850 4400 50  0001 C CNN
@@
 P 7900 5400
 F 0 "R8" V 7704 5400 50  0000 C CNN
-F 1 "10k" V 7795 5400 50  0000 C CNN
+F 1 "10K" V 7795 5400 50  0000 C CNN
 F 2 "Resistor_SMD:R_0603_1608Metric" H 7900 5400 50  0001 C CNN
 F 3 "~" H 7900 5400 50  0001 C CNN
@@
 P 7900 4000
 F 0 "R4" V 7704 4000 50  0000 C CNN
-F 1 "10k" V 7795 4000 50  0000 C CNN
+F 1 "10K" V 7795 4000 50  0000 C CNN
 F 2 "Resistor_SMD:R_0603_1608Metric" H 7900 4000 50  0001 C CNN
 F 3 "~" H 7900 4000 50  0001 C CNN
@@
 P 7900 5050
 F 0 "R7" V 7704 5050 50  0000 C CNN
-F 1 "10k" V 7795 5050 50  0000 C CNN
+F 1 "10K" V 7795 5050 50  0000 C CNN
 F 2 "Resistor_SMD:R_0603_1608Metric" H 7900 5050 50  0001 C CNN
 F 3 "~" H 7900 5050 50  0001 C CNN
@@
 P 7900 4350
 F 0 "R5" V 7704 4350 50  0000 C CNN
-F 1 "10k" V 7795 4350 50  0000 C CNN
+F 1 "10K" V 7795 4350 50  0000 C CNN
 F 2 "Resistor_SMD:R_0603_1608Metric" H 7900 4350 50  0001 C CNN
 F 3 "~" H 7900 4350 50  0001 C CNN
@@
 P 7900 4700
 F 0 "R6" V 7704 4700 50  0000 C CNN
-F 1 "10k" V 7795 4700 50  0000 C CNN
+F 1 "10K" V 7795 4700 50  0000 C CNN
 F 2 "Resistor_SMD:R_0603_1608Metric" H 7900 4700 50  0001 C CNN
 F 3 "~" H 7900 4700 50  0001 C CNN

Commit message: updated parts
Parts:
- C1: footprint Capacitor_Tantalum_SMD:CP_EIA-3216-18_Kemet-A -> Capacitor_Tantalum_SMD:CP_EIA-7343-31_Kemet-D; Supplier Part TPSA226K010R0900 -> T491D226K035AT
- C4: Supplier Part CL03B103KP3NNNC -> CL21B103KBANNNC
Changed lines of the file:
@@
 F 0 "C1" H 1838 1696 50  0000 L CNN
 F 1 "22uF" H 1838 1605 50  0000 L CNN
-F 2 "Capacitor_Tantalum_SMD:CP_EIA-3216-18_Kemet-A" H 1750 1650 50  0001 C CNN
+F 2 "Capacitor_Tantalum_SMD:CP_EIA-7343-31_Kemet-D" H 1750 1650 50  0001 C CNN
 F 3 "~" H 1750 1650 50  0001 C CNN
 F 4 "TME" H 1750 1650 50  0001 C CNN "Supplier"
-F 5 "TPSA226K010R0900" H 1750 1650 50  0001 C CNN "Supplier Part"
+F 5 "T491D226K035AT" H 1750 1650 50  0001 C CNN "Supplier Part"
 	1    1750 1650
 	1    0    0    -1
@@
 F 3 "~" H 2600 2550 50  0001 C CNN
 F 4 "TME" H 2600 2550 50  0001 C CNN "Supplier"
-F 5 "CL03B103KP3NNNC" H 2600 2550 50  0001 C CNN "Supplier Part"
+F 5 "CL21B103KBANNNC" H 2600 2550 50  0001 C CNN "Supplier Part"
 	1    2600 2550
 	1    0    0    -1

Commit message: reworked
- added correct circuit for BSS138
- added voltage divider for inputs
- changed buck converter setup
Parts:
- removed Q1, Q2: BSS138, Package_TO_SOT_SMD:SOT-23, symbol Device:Q_NPN_BCE
- added C2: 100nF, Capacitor_SMD:C_0603_1608Metric, symbol Device:C_Small
- added Q1, Q2: BSS138, Package_TO_SOT_SMD:SOT-23, symbol Transistor_FET:BSS138
- added R11, R12, R13, R14, R15: 100K, Resistor_SMD:R_0603_1608Metric, symbol Device:R_Small
- added R2, R3: 470R, Resistor_SMD:R_0603_1608Metric, symbol Device:R_Small
- added R4, R5: 4K7, Resistor_SMD:R_0603_1608Metric, symbol Device:R_Small
- C1: Supplier Part T491D226K035AT -> TAJD226K035R
- C3: renamed from C4; value 10nF -> 10uF; footprint Capacitor_SMD:C_0805_2012Metric -> Capacitor_SMD:C_0603_1608Metric; Supplier Part CL21B103KBANNNC -> CL10A106KQ8NNNC
- C4: renamed from C5; value 47uF -> 100nF; footprint Capacitor_SMD:C_0805_2012Metric -> Capacitor_SMD:C_0603_1608Metric; Supplier TM -> TME; Supplier Part CL21A476MQYNNNG -> CL10B104KO8NNNC
- C5: renamed from C2; value 0.01uF -> 10nF; Supplier Part 06035A100JAT2A -> CL10B103KB8NNNC
- L1: value 100uH -> 68uH; footprint Inductor_SMD:L_12x12mm_H8mm -> Inductor_SMD:L_12x12mm_H6mm; Supplier Part DE1207-120 -> DE1205-68
- R10: renamed from R8; value 10K -> 560K; Supplier Part SMD0603-10K-1% -> SMD0603-560K-1%
- R6: renamed from R4; value 10K -> 560K; Supplier Part SMD0603-10K-1% -> SMD0603-560K-1%
- R7: renamed from R5; value 10K -> 560K; Supplier Part SMD0603-10K-1% -> SMD0603-560K-1%
- R8: renamed from R6; value 10K -> 560K; Supplier Part SMD0603-10K-1% -> SMD0603-560K-1%
- R9: renamed from R7; value 10K -> 560K; Supplier Part SMD0603-10K-1% -> SMD0603-560K-1%
- renumbered C3 to C6, R2 to R1
Connections:
- net BTN_FANSPEED: now also Q2.3 (D)
- net BTN_POWER: now also Q1.3 (D)
- net GND: now also C2.2, Q1.2 (S), Q2.2 (S), R11.1, R12.1, R13.1, R14.1, R15.1, R4.1, R5.1
- net GPIO16: now also R3.2
- net GPIO17: now also R2.2
- net GPIO18: now also R15.2
- net GPIO19: now also R14.2
- net GPIO21: now also R13.2
- net GPIO22: now also R12.2
- net GPIO23: now also R11.2
- net RST: now also C2.1
- new net: Q1.1 (G), R2.1, R4.2
- new net: Q2.1 (G), R3.1, R5.2
Other:
- moved on the sheet: C1, C5, C6, D1, J2, L1, R1, R10, R6, R7, R8, R9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

Commit message: changed voltage divider to diodes
Parts:
- removed R10, R6, R7, R8, R9: 560K, Resistor_SMD:R_0603_1608Metric, symbol Device:R_Small
- removed R11, R12, R13, R14, R15: 100K, Resistor_SMD:R_0603_1608Metric, symbol Device:R_Small
- added D? (x5): 1N4148WS, Diode_SMD:D_SOD-323, symbol Diode:1N4148WS
Connections:
- net GPIO18: now also D?.2 (A)
- net GPIO19: now also D?.2 (A)
- net GPIO21: now also D?.2 (A)
- net GPIO22: now also D?.2 (A)
- net GPIO23: now also D?.2 (A)
- net LED_ERROR: now also D?.1 (K)
- net LED_HIGH: now also D?.1 (K)
- net LED_LOW: now also D?.1 (K)
- net LED_MID: now also D?.1 (K)
- net LED_POWER: now also D?.1 (K)
- no-connect marks 1 -> 23
