File: Venta LW Controller.sch (KiCad schematic (older format))
At the start: 26 parts, among them J1 Conn_01x04, J2 Conn_02x05_Odd_Even, Q1 BSS138, Q2 BSS138, SW1 RST, SW2 FLASH, U1 LM2674N-3.3, U2 ESP32-WROOM-32

Commit message: bumped version
Parts:
- gave numbers to parts that had none: 5
Changed lines of the file:
@@
 Title ""
 Date "2019-10-04"
-Rev "V2.1"
+Rev "V2.2"
 Comp ""
 Comment1 ""
@@
 	1450 950  1800 950
 $Comp
-L Diode:1N4148WS D?
+L Diode:1N4148WS D2
 U 1 1 5D9CF7F3
 P 9300 2150
-F 0 "D?" H 9300 2367 50  0000 C CNN
+F 0 "D2" H 9300 2367 50  0000 C CNN
 F 1 "1N4148WS" H 9300 2276 50  0000 C CNN
 F 2 "Diode_SMD:D_SOD-323" H 9300 1975 50  0001 C CNN
@@
 $EndComp
 $Comp
-L Diode:1N4148WS D?
+L Diode:1N4148WS D3
 U 1 1 5D9CFB7F
 P 9300 2800
-F 0 "D?" H 9300 3017 50  0000 C CNN
+F 0 "D3" H 9300 3017 50  0000 C CNN
 F 1 "1N4148WS" H 9300 2926 50  0000 C CNN
 F 2 "Diode_SMD:D_SOD-323" H 9300 2625 50  0001 C CNN
@@
 $EndComp
 $Comp
-L Diode:1N4148WS D?
+L Diode:1N4148WS D4
 U 1 1 5D9CFFBC
 P 9300 3500
-F 0 "D?" H 9300 3717 50  0000 C CNN
+F 0 "D4" H 9300 3717 50  0000 C CNN
 F 1 "1N4148WS" H 9300 3626 50  0000 C CNN
 F 2 "Diode_SMD:D_SOD-323" H 9300 3325 50  0001 C CNN
@@
 $EndComp
 $Comp
-L Diode:1N4148WS D?
+L Diode:1N4148WS D5
 U 1 1 5D9D0425
 P 9300 4150
-F 0 "D?" H 9300 4367 50  0000 C CNN
+F 0 "D5" H 9300 4367 50  0000 C CNN
 F 1 "1N4148WS" H 9300 4276 50  0000 C CNN
 F 2 "Diode_SMD:D_SOD-323" H 9300 3975 50  0001 C CNN
@@
 $EndComp
 $Comp
-L Diode:1N4148WS D?
+L Diode:1N4148WS D6
 U 1 1 5D9D0838
 P 9300 4800
-F 0 "D?" H 9300 5017 50  0000 C CNN
+F 0 "D6" H 9300 5017 50  0000 C CNN
 F 1 "1N4148WS" H 9300 4926 50  0000 C CNN
 F 2 "Diode_SMD:D_SOD-323" H 9300 4625 50  0001 C CNN

Commit message: refilled and rotated connector
Connections:
- net +24V: now also J2.1 (Pin_1); no longer J2.10 (Pin_10)
- net BTN_COVER: now also J2.5 (Pin_5); no longer J2.6 (Pin_6)
- net BTN_FANSPEED: now also J2.9 (Pin_9); no longer J2.2 (Pin_2)
- net BTN_POWER: now also J2.7 (Pin_7); no longer J2.4 (Pin_4)
- net GND: now also J2.3 (Pin_3); no longer J2.8 (Pin_8)
- net LED_ERROR: now also J2.10 (Pin_10); no longer J2.1 (Pin_1)
- net LED_HIGH: now also J2.8 (Pin_8); no longer J2.3 (Pin_3)
- net LED_LOW: now also J2.4 (Pin_4); no longer J2.7 (Pin_7)
- net LED_MID: now also J2.6 (Pin_6); no longer J2.5 (Pin_5)
- net LED_POWER: now also J2.2 (Pin_2); no longer J2.9 (Pin_9)
Changed lines of the file:
@@
 EESchema Schematic File Version 4
-LIBS:Venta LW Controller-cache
 EELAYER 30 0
 EELAYER END
@@
 Text GLabel 5100 6650 0    50   Input ~ 0
 LED_ERROR
-Wire Wire Line
-	5100 6650 5350 6650
-Wire Wire Line
-	5100 6750 5350 6750
-Wire Wire Line
-	5350 6850 5100 6850
-Wire Wire Line
-	5100 6950 5350 6950
-Wire Wire Line
-	5850 6650 6100 6650
-Wire Wire Line
-	6100 6750 5850 6750
-Wire Wire Line
-	6100 6950 5850 6950
-Wire Wire Line
-	5850 7050 6100 7050
 Text GLabel 6100 6850 2    50   Input ~ 0
 BTN_COVER
 Wire Wire Line
-	5100 7050 5350 7050
-Wire Wire Line
 	1450 1700 2300 1700
-$Comp
-L Connector_Generic:Conn_02x05_Odd_Even J2
-U 1 1 5D7A19E5
-P 5550 6850
-F 0 "J2" H 5600 7267 50  0000 C CNN
-F 1 "Conn_02x05_Odd_Even" H 5600 7176 50  0000 C CNN
-F 2 "Connector_IDC:IDC-Header_2x05_P2.54mm_Vertical" H 5550 6850 50  0001 C CNN
-F 3 "~" H 5550 6850 50  0001 C CNN
-F 4 "TME" H 5550 6850 50  0001 C CNN "Supplier"
-F 5 "T821-1-10-S1" H 5550 6850 50  0001 C CNN "Supplier Part"
-	1    5550 6850
-	1    0    0    -1
-$EndComp
 Text GLabel 4450 4400 2    50   Input ~ 0
 GPIO18
@@
 NoConn ~ 4350 3400
 Wire Wire Line
-	5850 6850 6100 6850
-Wire Wire Line
 	1450 950  1800 950
 $Comp
@@
 Wire Wire Line
 	9450 4800 9750 4800
+Wire Wire Line
+	5100 6650 5350 6650
+Wire Wire Line
+	5100 6750 5350 6750
+Wire Wire Line
+	5100 6850 5350 6850
+Wire Wire Line
+	5100 6950 5350 6950
+Wire Wire Line
+	5100 7050 5350 7050
+Wire Wire Line
+	5850 6650 6100 6650
+Wire Wire Line
+	6100 6750 5850 6750
+Wire Wire Line
+	5850 6850 6100 6850
+Wire Wire Line
+	6100 6950 5850 6950
+Wire Wire Line
+	5850 7050 6100 7050
+$Comp
+L Connector_Generic:Conn_02x05_Odd_Even J2
+U 1 1 5D7A19E5
+P 5650 6850
+F 0 "J2" H 5700 7267 50  0000 C CNN
+F 1 "Conn_02x05_Odd_Even" H 5700 7176 50  0000 C CNN
+F 2 "Connector_IDC:IDC-Header_2x05_P2.54mm_Vertical" H 5650 6850 50  0001 C CNN
+F 3 "~" H 5650 6850 50  0001 C CNN
+F 4 "TME" H 5650 6850 50  0001 C CNN "Supplier"
+F 5 "T821-1-10-S1" H 5650 6850 50  0001 C CNN "Supplier Part"
+	1    5650 6850
+	-1   0    0    1
+$EndComp
 $EndSCHEMATC
