File: Venta LW Controller.kicad_pcb (KiCad board)
At the start: 2 copper layers, 56 x 99.2 mm, 29 parts, among them J1 Conn_01x04, J2 Conn_02x05_Odd_Even, Q1 BSS138, Q2 BSS138, SW1 RST, SW2 FLASH, U1 LM2674N-3.3, U2 ESP-12F

Commit message: use usable GPIOs
Parts:
- C1: value 25u -> 22u
- C5: value 100u -> 47u
Connections:
- J1 pad 3: RXD -> GPIO3
- J1 pad 4: TXD -> GPIO1
- R4 pad 1: GPIO7 -> GPIO13
- R5 pad 1: GPIO9 -> GPIO12
- R6 pad 1: GPIO10 -> GPIO14
- R7 pad 1: GPIO8 -> GPIO1
- R8 pad 1: GPIO6 -> GPIO3
- U2 pad 15: RXD -> GPIO3
- U2 pad 16: TXD -> GPIO1
- U2 pad 18: GPIO7 -> Net-(U2-Pad18)
- U2 pad 19: GPIO9 -> Net-(U2-Pad19)
- U2 pad 20: GPIO10 -> Net-(U2-Pad20)
- U2 pad 21: GPIO8 -> Net-(U2-Pad21)
- U2 pad 22: GPIO6 -> Net-(U2-Pad22)
- U2 pad 5: Net-(U2-Pad5) -> GPIO14
- U2 pad 6: Net-(U2-Pad6) -> GPIO12
- U2 pad 7: Net-(U2-Pad7) -> GPIO13
Routing:
- net GPIO1: track 0.00 -> 80.8 mm, vias 0 -> 2
- net GPIO3: track 0.00 -> 78.7 mm
- net TXD: track 61.4 -> 0.00 mm
- net RXD: track 59.9 -> 0.00 mm
- net GPIO14: track 0.00 -> 14.4 mm
- net GPIO12: track 0.00 -> 11.5 mm
- net GPIO13: track 0.00 -> 8.69 mm
- net FLASH: track 94.3 -> 88.5 mm
- net GPIO6: track 3.66 -> 0.00 mm
- net GPIO10: track 3.65 -> 0.00 mm
- net GPIO9: track 3.65 -> 0.00 mm
- net GPIO8: track 3.65 -> 0.00 mm
- net GPIO7: track 3.65 -> 0.00 mm

Commit message: bumped version
Other:
- board text added: "ALITECS Venta LW Controller V1.1"
- board text removed: "ALITECS Venta LW Controller V1.0"
Changed lines of the file:
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@@
     )
   )
-  (gr_text "ALITECS\nVenta LW Controller\nV1.0" (at 125.75 48.85) (layer F.SilkS)
+  (gr_text "ALITECS\nVenta LW Controller\nV1.1" (at 125.75 48.85) (layer F.SilkS)
     (effects (font (size 1 1) (thickness 0.15)) (justify left))
   )

Commit message: updated tracks
Routing:
- net FLASH: track 88.5 -> 89.2 mm
Changed lines of the file:
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@@
     (thickness 1.6)
     (drawings 32)
-    (tracks 197)
+    (tracks 198)
     (zones 0)
     (modules 29)
@@
   (segment (start 148.149919 86.095083) (end 148.149919 94.149919) (width 0.25) (layer B.Cu) (net 6))
   (segment (start 148.14999 76.94249) (end 148.14999 86.095012) (width 0.25) (layer B.Cu) (net 6))
-  (segment (start 129.338 77.55) (end 129.384 77.504) (width 0.25) (layer B.Cu) (net 28) (status 30))
-  (segment (start 151.18 110.85) (end 129.263589 110.85) (width 0.25) (layer B.Cu) (net 28) (status 10))
-  (segment (start 125.308955 106.895366) (end 125.308955 79.441045) (width 0.25) (layer B.Cu) (net 28))
-  (segment (start 129.263589 110.85) (end 125.308955 106.895366) (width 0.25) (layer B.Cu) (net 28))
-  (segment (start 125.308955 79.441045) (end 127.2 77.55) (width 0.25) (layer B.Cu) (net 28))
-  (segment (start 151.2 110.87) (end 151.18 110.85) (width 0.25) (layer B.Cu) (net 28) (status 30))
-  (segment (start 127.2 77.55) (end 129.338 77.55) (width 0.25) (layer B.Cu) (net 28) (status 20))
-  (segment (start 163.34 103) (end 136.846504 103) (width 0.25) (layer F.Cu) (net 7) (status 10))
-  (segment (start 136.846504 103) (end 131.782499 97.935995) (width 0.25) (layer F.Cu) (net 7))
   (via (at 131.3825 97.535996) (size 0.8) (drill 0.4) (layers F.Cu B.Cu) (net 7))
-  (segment (start 131.782499 97.935995) (end 131.3825 97.535996) (width 0.25) (layer F.Cu) (net 7))
   (segment (start 131.3825 96.970311) (end 131.3825 97.535996) (width 0.25) (layer B.Cu) (net 7))
   (segment (start 131.39 95.7072) (end 131.3825 95.7147) (width 0.25) (layer B.Cu) (net 7) (status 30))
   (segment (start 131.3825 95.7147) (end 131.3825 96.970311) (width 0.25) (layer B.Cu) (net 7) (status 10))
+  (segment (start 135.268704 101.4222) (end 131.782499 97.935995) (width 0.25) (layer F.Cu) (net 7))
+  (segment (start 131.782499 97.935995) (end 131.3825 97.535996) (width 0.25) (layer F.Cu) (net 7))
+  (segment (start 163.34 103) (end 161.7622 101.4222) (width 0.25) (layer F.Cu) (net 7))
+  (segment (start 161.7622 101.4222) (end 135.268704 101.4222) (width 0.25) (layer F.Cu) (net 7))
   (via (at 133.349996 97.536) (size 0.8) (drill 0.4) (layers F.Cu B.Cu) (net 8))
   (segment (start 136.785395 100.971399) (end 133.749995 97.935999) (width 0.25) (layer F.Cu) (net 8))
@@
   (segment (start 139.3952 97.536) (end 141.478 99.6188) (width 0.25) (layer F.Cu) (net 11))
   (segment (start 141.478 99.6188) (end 170.0784 99.6188) (width 0.25) (layer F.Cu) (net 11))
-  (segment (start 133.934 102.632) (end 136.654011 105.352011) (width 0.25) (layer B.Cu) (net 13))
-  (segment (start 172.636401 106.403599) (end 173.5 105.54) (width 0.25) (layer B.Cu) (net 13) (status 20))
-  (segment (start 133.284 102.632) (end 133.934 102.632) (width 0.25) (layer B.Cu) (net 13) (status 10))
+  (segment (start 172.636401 106.403599) (end 173.5 105.54) (width 0.25) (layer B.Cu) (net 13))
+  (segment (start 133.284 102.632) (end 133.934 102.632) (width 0.25) (layer B.Cu) (net 13))
+  (segment (start 136.839 105.537) (end 161.6425 105.537) (width 0.25) (layer B.Cu) (net 13))
   (segment (start 162.834101 106.728601) (end 172.311399 106.728601) (width 0.25) (layer B.Cu) (net 13))
-  (segment (start 136.654011 105.352011) (end 161.457511 105.352011) (width 0.25) (layer B.Cu) (net 13))
-  (segment (start 161.457511 105.352011) (end 162.834101 106.728601) (width 0.25) (layer B.Cu) (net 13))
+  (segment (start 133.934 102.632) (end 136.839 105.537) (width 0.25) (layer B.Cu) (net 13))
+  (segment (start 161.6425 105.537) (end 162.834101 106.728601) (width 0.25) (layer B.Cu) (net 13))
   (segment (start 172.311399 106.728601) (end 172.636401 106.403599) (width 0.25) (layer B.Cu) (net 13))
   (segment (start 170.096401 104.676401) (end 170.96 105.54) (width 0.25) (layer B.Cu) (net 14) (status 20))
@@
   (segment (start 162.99 111.77) (end 165.032 109.728) (width 0.25) (layer B.Cu) (net 19) (status 10))
   (via (at 131.375667 83.4898) (size 0.8) (drill 0.4) (layers F.Cu B.Cu) (net 19))
-  (segment (start 131.941352 83.4898) (end 131.375667 83.4898) (width 0.25) (layer F.Cu) (net 19))
-  (segment (start 147.574012 94.354127) (end 136.709685 83.4898) (width 0.25) (layer F.Cu) (net 19))
-  (segment (start 136.709685 83.4898) (end 131.941352 83.4898) (width 0.25) (layer F.Cu) (net 19))
-  (segment (start 147.574012 97.536) (end 147.574012 94.354127) (width 0.25) (layer F.Cu) (net 19))
   (segment (start 130.809982 83.4898) (end 131.375667 83.4898) (width 0.25) (layer B.Cu) (net 19))
   (segment (start 129.3982 83.4898) (end 130.809982 83.4898) (width 0.25) (layer B.Cu) (net 19))
   (segment (start 129.384 83.504) (end 129.3982 83.4898) (width 0.25) (layer B.Cu) (net 19))
+  (segment (start 137.922 83.4898) (end 131.941352 83.4898) (width 0.25) (layer F.Cu) (net 19))
+  (segment (start 147.574012 97.536) (end 147.574012 93.141812) (width 0.25) (layer F.Cu) (net 19))
+  (segment (start 131.941352 83.4898) (end 131.375667 83.4898) (width 0.25) (layer F.Cu) (net 19))
+  (segment (start 147.574012 93.141812) (end 137.922 83.4898) (width 0.25) (layer F.Cu) (net 19))
   (via (at 126.187198 105.5624) (size 0.8) (drill 0.4) (layers F.Cu B.Cu) (net 27))
   (segment (start 151.2 108.33) (end 128.954798 108.33) (width 0.25) (layer B.Cu) (net 27))
@@
   (segment (start 126.187198 75.539644) (end 126.187221 75.539621) (width 0.25) (layer F.Cu) (net 27))
   (segment (start 126.187198 105.5624) (end 126.187198 75.539644) (width 0.25) (layer F.Cu) (net 27))
+  (segment (start 134.3914 79.8068) (end 130.0886 75.504) (width 0.25) (layer B.Cu) (net 27))
+  (segment (start 134.3914 92.6086) (end 134.3914 79.8068) (width 0.25) (layer B.Cu) (net 27))
   (segment (start 130.0886 75.504) (end 129.384 75.504) (width 0.25) (layer B.Cu) (net 27))
-  (segment (start 134.269001 79.684401) (end 130.0886 75.504) (width 0.25) (layer B.Cu) (net 27))
-  (segment (start 134.269001 92.730999) (end 134.269001 79.684401) (width 0.25) (layer B.Cu) (net 27))
   (segment (start 133.39 94.1475) (end 133.39 93.61) (width 0.25) (layer B.Cu) (net 27))
-  (segment (start 133.39 93.61) (end 134.269001 92.730999) (width 0.25) (layer B.Cu) (net 27))
-  (segment (start 132.518999 79.991799) (end 130.0312 77.504) (width 0.25) (layer B.Cu) (net 28))
-  (segment (start 131.39 94.1577) (end 132.518999 93.028701) (width 0.25) (layer B.Cu) (net 28))
+  (segment (start 133.39 93.61) (end 134.3914 92.6086) (width 0.25) (layer B.Cu) (net 27))
+  (segment (start 129.338 77.55) (end 129.384 77.504) (width 0.25) (layer B.Cu) (net 28) (status 30))
+  (segment (start 151.18 110.85) (end 129.263589 110.85) (width 0.25) (layer B.Cu) (net 28) (status 10))
+  (segment (start 125.308955 106.895366) (end 125.308955 79.441045) (width 0.25) (layer B.Cu) (net 28))
+  (segment (start 129.263589 110.85) (end 125.308955 106.895366) (width 0.25) (layer B.Cu) (net 28))
+  (segment (start 125.308955 79.441045) (end 127.2 77.55) (width 0.25) (layer B.Cu) (net 28))
+  (segment (start 151.2 110.87) (end 151.18 110.85) (width 0.25) (layer B.Cu) (net 28) (status 30))
+  (segment (start 127.2 77.55) (end 129.338 77.55) (width 0.25) (layer B.Cu) (net 28) (status 20))
   (segment (start 130.0312 77.504) (end 129.384 77.504) (width 0.25) (layer B.Cu) (net 28))
-  (segment (start 132.518999 93.028701) (end 132.518999 79.991799) (width 0.25) (layer B.Cu) (net 28))
+  (segment (start 131.39 94.1577) (end 132.3848 93.1629) (width 0.25) (layer B.Cu) (net 28))
+  (segment (start 132.3848 79.8576) (end 130.0312 77.504) (width 0.25) (layer B.Cu) (net 28))
+  (segment (start 132.3848 93.1629) (end 132.3848 79.8576) (width 0.25) (layer B.Cu) (net 28))
   (segment (start 142.708998 83.504) (end 143.384 83.504) (width 0.25) (layer B.Cu) (net 29))
   (segment (start 136.3726 89.840398) (end 142.708998 83.504) (width 0.25) (layer B.Cu) (net 29))

Commit message: updated layout
Parts:
- R4, R5, R6, R7, R8: moved to F.Cu
- moved C1 23.8 mm to (151.0, 124.2), turned to 270 degrees
- moved D1 16.5 mm to (153.4, 120.0)
- moved U1 15.0 mm to (144.4, 124.1), turned to 0 degrees
- moved C2 10.2 mm to (144.4, 117.8)
- moved L1 8.65 mm to (131.8, 125.6)
- moved R3 8.64 mm to (126.1, 86.7)
- moved R2 6.82 mm to (146.5, 87.1)
- moved C3 3.36 mm to (143.1, 131.6)
- moved U2 1.59 mm to (143.2, 73.9)
- moved R1 1.56 mm to (146.5, 74.7)
- moved SW1 0.97 mm to (169.6, 111.8)
- moved SW2 0.97 mm to (157.5, 111.8)
- moved J1 0.54 mm to (151.7, 116.0)
- turned Q2 to 0 degrees
Connections:
- C3 pad 1: Net-(C2-Pad2) -> +3.3V
- U1 pad 4: Net-(C2-Pad2) -> +3.3V
Routing:
- net FLASH: track 89.2 -> 57.0 mm, vias 2 -> 1
- net +24V: track 51.6 -> 28.7 mm, vias 2 -> 0
- net +3.3V: track 75.9 -> 84.6 mm
- net Net-(R2-Pad2): track 3.32 -> 10.4 mm
- net GPIO1: track 80.9 -> 86.9 mm, vias 2 -> 3
- net Net-(R3-Pad2): track 8.87 -> 3.15 mm
- net Net-(C2-Pad2): track 32.1 -> 37.2 mm
- net GPIO5: track 27.8 -> 32.8 mm
- net GPIO4: track 32.0 -> 28.6 mm
- net BTN_FANSPEED: track 42.4 -> 45.5 mm, vias 0 -> 1
- net GPIO14: track 14.4 -> 16.6 mm, vias 0 -> 1
- net GPIO12: track 11.5 -> 13.8 mm, vias 0 -> 1
- net GPIO13: track 8.69 -> 10.9 mm, vias 0 -> 1
- net Net-(C2-Pad1): track 3.02 -> 4.65 mm
- net BTN_POWER: track 34.9 -> 36.4 mm
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
Commit message: updated package
Parts:
- U1: footprint Package_DIP:DIP-8_W7.62mm_SMDSocket_SmallPads -> Package_SO:SOIC-8_3.9x4.9mm_P1.27mm
- moved L1 5.38 mm to (131.7, 131.0)
- moved C3 2.82 mm to (144.4, 129.1)
- moved C2 2.61 mm to (144.4, 120.4)
- moved C1 0.62 mm to (150.9, 124.9)
Routing:
- net Net-(C2-Pad2): track 37.2 -> 33.5 mm
- net Net-(C2-Pad1): track 4.65 -> 2.51 mm
- net +3.3V: track 84.6 -> 82.5 mm
- net +24V: track 28.7 -> 30.2 mm

Commit message: bumped version
Other:
- board text added: "ALITECS Venta LW Controller V1.2"
- board text removed: "ALITECS Venta LW Controller V1.1"
Changed lines of the file:
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@@
     )
   )
-  (gr_text "ALITECS\nVenta LW Controller\nV1.1" (at 125.75 48.85) (layer F.SilkS)
+  (gr_text "ALITECS\nVenta LW Controller\nV1.2" (at 125.75 48.85) (layer F.SilkS)
     (effects (font (size 1 1) (thickness 0.15)) (justify left))
   )
