File: Venta LW Controller.kicad_pcb (KiCad board)
At the start: 2 copper layers, 56 x 99.2 mm, 29 parts, among them J1 Conn_01x04, J2 Conn_02x05_Odd_Even, Q1 BSS138, Q2 BSS138, SW1 RST, SW2 FLASH, U1 LM2674N-3.3, U2 ESP-12F

Commit message: switched to ESP32
Parts:
- removed C7: 100n, Capacitor_SMD:C_0805_2012Metric
- removed R1, R3: 10k, Resistor_SMD:R_0603_1608Metric
- U2: value ESP-12F -> ESP32-WROOM-32; footprint ALITECS:ESP-12E -> RF_Module:ESP32-WROOM-32
- moved U2 9.00 mm to (136.4, 81.2)
- moved R2 0.62 mm to (147.3, 80.1)
Connections:
- J1 pad 3: GPIO3 -> RXD
- J1 pad 4: GPIO1 -> TXD
- Q1 pad 1: GPIO4 -> GPIO17
- Q2 pad 1: GPIO5 -> GPIO16
- R2 pad 2: Net-(R2-Pad2) -> RST
- R4 pad 1: GPIO13 -> GPIO23
- R5 pad 1: GPIO12 -> GPIO22
- R6 pad 1: GPIO14 -> GPIO21
- R7 pad 1: GPIO1 -> GPIO19
- R8 pad 1: GPIO3 -> GPIO18
- U2 pad 1: RST -> GND
- U2 pad 12: FLASH -> Net-(U2-Pad12)
- U2 pad 13: GPIO4 -> Net-(U2-Pad13)
- U2 pad 14: GPIO5 -> Net-(U2-Pad14)
- U2 pad 15: GPIO3 -> GND
- U2 pad 16: GPIO1 -> Net-(U2-Pad16)
- U2 pad 2: Net-(U2-Pad2) -> +3.3V
- U2 pad 3: Net-(R2-Pad2) -> RST
- U2 pad 5: GPIO14 -> Net-(U2-Pad5)
- U2 pad 6: GPIO12 -> Net-(U2-Pad6)
- U2 pad 7: GPIO13 -> Net-(U2-Pad7)
- U2 pad 8: +3.3V -> Net-(U2-Pad8)
- U2 pad 9: GND -> Net-(U2-Pad9)
Routing:
- net GPIO1: track 80.8 -> 0.00 mm, vias 2 -> 0
- net GPIO3: track 78.7 -> 0.00 mm
- net RXD: track 0.00 -> 53.3 mm
- net TXD: track 0.00 -> 52.7 mm, vias 0 -> 2
- net FLASH: track 88.5 -> 49.0 mm
- net GPIO4: track 32.0 -> 0.00 mm
- net GPIO23: track 0.00 -> 28.3 mm, vias 0 -> 2
- net GPIO5: track 27.8 -> 0.00 mm
- net GPIO22: track 0.00 -> 25.8 mm, vias 0 -> 2
- net GPIO17: track 0.00 -> 23.6 mm
- net GPIO21: track 0.00 -> 20.6 mm, vias 0 -> 2
- net GPIO16: track 0.00 -> 17.9 mm
- net GPIO19: track 0.00 -> 16.9 mm, vias 0 -> 2
- net GPIO14: track 14.4 -> 0.00 mm
- net GPIO18: track 0.00 -> 14.3 mm, vias 0 -> 2
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
Commit message: corrected circuit and updated layout
Parts:
- R4, R5, R6, R7, R8: moved to F.Cu
- moved C1 23.8 mm to (151.0, 124.2), turned to 270 degrees
- moved D1 16.5 mm to (153.4, 120.0)
- moved U1 15.0 mm to (144.4, 124.1), turned to 0 degrees
- moved C2 10.2 mm to (144.4, 117.8)
- moved L1 8.65 mm to (131.8, 125.6)
- moved C3 3.36 mm to (143.1, 131.6)
- moved SW1 0.97 mm to (169.6, 111.8)
- moved SW2 0.97 mm to (157.5, 111.8)
- moved J1 0.54 mm to (151.7, 116.0)
Connections:
- C3 pad 1: Net-(C2-Pad2) -> +3.3V
- U1 pad 4: Net-(C2-Pad2) -> +3.3V
Routing:
- net +24V: track 51.6 -> 28.7 mm, vias 2 -> 0
- net +3.3V: track 68.0 -> 84.6 mm
- net Net-(C2-Pad2): track 32.1 -> 37.2 mm
- net Net-(C2-Pad1): track 3.02 -> 4.65 mm
- net FLASH: track 49.0 -> 50.6 mm
- net RXD: track 53.3 -> 53.8 mm
- net TXD: track 52.7 -> 53.3 mm
- net LED_ERROR: track 38.5 -> 38.2 mm, vias 1 -> 0
- net GPIO19: track 16.9 -> 16.8 mm, vias 2 -> 1
- net LED_LOW: vias 1 -> 0
- net LED_POWER: track 36.1 -> 36.0 mm, vias 1 -> 0
- net LED_MID: vias 1 -> 0
- net LED_HIGH: vias 1 -> 0
- net GPIO18: vias 2 -> 1
- net GPIO23: vias 2 -> 1
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
Commit message: updated layout
Routing:
- net RST: track 79.4 -> 81.7 mm
- net RXD: track 53.8 -> 55.4 mm, vias 0 -> 2
- net TXD: track 53.3 -> 52.7 mm
- net BTN_FANSPEED: track 42.4 -> 42.2 mm, vias 0 -> 1
- net GND: vias 6 -> 3
Changed lines of the file:
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@@
     (thickness 1.6)
     (drawings 32)
-    (tracks 172)
+    (tracks 174)
     (zones 0)
     (modules 26)
@@
   (gr_line (start 148.5 52.76) (end 148.5 95.5) (layer Edge.Cuts) (width 0.05))
   (gr_arc (start 119 91) (end 127.499616 42.430432) (angle 25.3818742) (layer Edge.Cuts) (width 0.05))
-  (via (at 145.2372 98.1202) (size 0.8) (drill 0.4) (layers F.Cu B.Cu) (net 1))
-  (via (at 140.843 88.1634) (size 0.8) (drill 0.4) (layers F.Cu B.Cu) (net 1))
-  (via (at 142.5448 72.9488) (size 0.8) (drill 0.4) (layers F.Cu B.Cu) (net 1))
-  (via (at 130.6068 72.9488) (size 0.8) (drill 0.4) (layers F.Cu B.Cu) (net 1))
-  (via (at 140.8684 103.6066) (size 0.8) (drill 0.4) (layers F.Cu B.Cu) (net 1))
-  (via (at 133.3246 105.918) (size 0.8) (drill 0.4) (layers F.Cu B.Cu) (net 1))
+  (via (at 142.113 72.94372) (size 0.8) (drill 0.4) (layers F.Cu B.Cu) (net 1))
+  (via (at 130.08864 72.95388) (size 0.8) (drill 0.4) (layers F.Cu B.Cu) (net 1))
+  (via (at 142.12824 92.49664) (size 0.8) (drill 0.4) (layers F.Cu B.Cu) (net 1))
   (segment (start 150.9804 122.8715) (end 151.003 122.8941) (width 0.25) (layer F.Cu) (net 2))
   (segment (start 148.2102 122.8715) (end 150.9804 122.8715) (width 0.25) (layer F.Cu) (net 2))
@@
   (segment (start 174.720987 111.77) (end 169.6352 111.77) (width 0.25) (layer B.Cu) (net 6))
   (segment (start 176.1352 111.77) (end 174.720987 111.77) (width 0.25) (layer B.Cu) (net 6))
+  (segment (start 149.810409 98.350009) (end 146.932599 95.472199) (width 0.25) (layer B.Cu) (net 6))
   (segment (start 146.932599 95.472199) (end 146.5326 95.0722) (width 0.25) (layer B.Cu) (net 6))
-  (segment (start 173.94182 98.350009) (end 149.810409 98.350009) (width 0.25) (layer B.Cu) (net 6))
-  (segment (start 176.169999 100.578188) (end 173.94182 98.350009) (width 0.25) (layer B.Cu) (net 6))
-  (segment (start 149.810409 98.350009) (end 146.932599 95.472199) (width 0.25) (layer B.Cu) (net 6))
-  (segment (start 176.1352 111.77) (end 176.169999 111.735201) (width 0.25) (layer B.Cu) (net 6))
-  (segment (start 176.169999 111.735201) (end 176.169999 100.578188) (width 0.25) (layer B.Cu) (net 6))
+  (segment (start 177.6476 100.16744) (end 175.830169 98.350009) (width 0.25) (layer B.Cu) (net 6))
+  (segment (start 175.830169 98.350009) (end 149.810409 98.350009) (width 0.25) (layer B.Cu) (net 6))
+  (segment (start 176.1352 111.77) (end 177.6476 110.2576) (width 0.25) (layer B.Cu) (net 6))
+  (segment (start 177.6476 110.2576) (end 177.6476 100.16744) (width 0.25) (layer B.Cu) (net 6))
   (via (at 136.906 108.3056) (size 0.8) (drill 0.4) (layers F.Cu B.Cu) (net 7))
-  (via (at 125.67922 76.7588) (size 0.8) (drill 0.4) (layers F.Cu B.Cu) (net 7))
-  (segment (start 127.9234 76.7588) (end 125.67922 76.7588) (width 0.25) (layer B.Cu) (net 7))
-  (segment (start 136.906 108.3056) (end 125.67922 97.07882) (width 0.25) (layer F.Cu) (net 7))
-  (segment (start 125.67922 77.324485) (end 125.67922 76.7588) (width 0.25) (layer F.Cu) (net 7))
-  (segment (start 125.67922 97.07882) (end 125.67922 77.324485) (width 0.25) (layer F.Cu) (net 7))
   (segment (start 136.9304 108.33) (end 136.906 108.3056) (width 0.25) (layer B.Cu) (net 7))
   (segment (start 151.7396 108.3564) (end 151.7132 108.33) (width 0.25) (layer B.Cu) (net 7))
   (segment (start 151.7132 108.33) (end 136.9304 108.33) (width 0.25) (layer B.Cu) (net 7))
-  (segment (start 126.6734 78.0288) (end 127.9234 78.0288) (width 0.25) (layer B.Cu) (net 8))
-  (segment (start 125.698379 79.003821) (end 126.6734 78.0288) (width 0.25) (layer B.Cu) (net 8))
-  (segment (start 125.698379 99.431381) (end 125.698379 79.003821) (width 0.25) (layer B.Cu) (net 8))
-  (segment (start 137.136998 110.87) (end 125.698379 99.431381) (width 0.25) (layer B.Cu) (net 8))
-  (segment (start 151.7396 110.8964) (end 151.7132 110.87) (width 0.25) (layer B.Cu) (net 8))
-  (segment (start 151.7132 110.87) (end 137.136998 110.87) (width 0.25) (layer B.Cu) (net 8))
+  (via (at 126.11608 76.758804) (size 0.8) (drill 0.4) (layers F.Cu B.Cu) (net 7))
+  (segment (start 136.906 108.3056) (end 126.11608 97.51568) (width 0.25) (layer F.Cu) (net 7))
+  (segment (start 127.9234 76.7588) (end 126.116084 76.7588) (width 0.25) (layer B.Cu) (net 7))
+  (segment (start 126.11608 97.51568) (end 126.11608 77.324489) (width 0.25) (layer F.Cu) (net 7))
+  (segment (start 126.116084 76.7588) (end 126.11608 76.758804) (width 0.25) (layer B.Cu) (net 7))
+  (segment (start 126.11608 77.324489) (end 126.11608 76.758804) (width 0.25) (layer F.Cu) (net 7))
+  (segment (start 125.150412 78.0288) (end 125.125012 78.0542) (width 0.25) (layer B.Cu) (net 8))
+  (via (at 125.125012 78.0542) (size 0.8) (drill 0.4) (layers F.Cu B.Cu) (net 8))
+  (segment (start 127.9234 78.0288) (end 125.150412 78.0288) (width 0.25) (layer B.Cu) (net 8))
+  (via (at 136.906 110.896402) (size 0.8) (drill 0.4) (layers F.Cu B.Cu) (net 8))
+  (segment (start 151.7396 110.8964) (end 136.906002 110.8964) (width 0.25) (layer B.Cu) (net 8))
+  (segment (start 136.906002 110.8964) (end 136.906 110.896402) (width 0.25) (layer B.Cu) (net 8))
+  (segment (start 125.125012 78.0542) (end 125.125012 99.115414) (width 0.25) (layer F.Cu) (net 8))
+  (segment (start 136.506001 110.496403) (end 136.906 110.896402) (width 0.25) (layer F.Cu) (net 8))
+  (segment (start 125.125012 99.115414) (end 136.506001 110.496403) (width 0.25) (layer F.Cu) (net 8))
   (segment (start 135.268704 101.4222) (end 131.39 97.543496) (width 0.25) (layer F.Cu) (net 9))
   (segment (start 131.39 97.543496) (end 131.39 95.7327) (width 0.25) (layer F.Cu) (net 9))
   (segment (start 163.34 103) (end 161.7622 101.4222) (width 0.25) (layer F.Cu) (net 9))
   (segment (start 161.7622 101.4222) (end 135.268704 101.4222) (width 0.25) (layer F.Cu) (net 9))
-  (segment (start 133.35 95.7072) (end 133.349996 95.707204) (width 0.25) (layer B.Cu) (net 10) (status 30))
-  (segment (start 133.39 97.495996) (end 133.39 95.7225) (width 0.25) (layer F.Cu) (net 10))
-  (segment (start 133.39 97.576004) (end 133.39 97.495996) (width 0.25) (layer F.Cu) (net 10))
+  (segment (start 133.39 97.576004) (end 133.39 95.7225) (width 0.25) (layer F.Cu) (net 10))
   (segment (start 136.785395 100.971399) (end 133.39 97.576004) (width 0.25) (layer F.Cu) (net 10))
   (segment (start 165.88 103) (end 163.851399 100.971399) (width 0.25) (layer F.Cu) (net 10))
@@
   (segment (start 173.4596 103) (end 170.0784 99.6188) (width 0.25) (layer F.Cu) (net 13))
   (segment (start 133.934 102.632) (end 136.654011 105.352011) (width 0.25) (layer B.Cu) (net 15))
-  (segment (start 172.311399 106.728601) (end 173.5 105.54) (width 0.25) (layer B.Cu) (net 15) (status 20))
   (segment (start 133.284 102.632) (end 133.934 102.632) (width 0.25) (layer B.Cu) (net 15) (status 10))
-  (segment (start 162.834101 106.728601) (end 172.311399 106.728601) (width 0.25) (layer B.Cu) (net 15))
   (segment (start 136.654011 105.352011) (end 161.457511 105.352011) (width 0.25) (layer B.Cu) (net 15))
-  (segment (start 161.457511 105.352011) (end 162.834101 106.728601) (width 0.25) (layer B.Cu) (net 15))
+  (segment (start 161.457511 105.352011) (end 161.457511 105.352011) (width 0.25) (layer B.Cu) (net 15))
+  (via (at 161.457511 105.352011) (size 0.8) (drill 0.4) (layers F.Cu B.Cu) (net 15))
+  (segment (start 172.636401 104.676401) (end 173.5 105.54) (width 0.25) (layer F.Cu) (net 15))
+  (segment (start 172.311399 104.351399) (end 172.636401 104.676401) (width 0.25) (layer F.Cu) (net 15))
+  (segment (start 161.457511 105.352011) (end 162.458123 104.351399) (width 0.25) (layer F.Cu) (net 15))
+  (segment (start 162.458123 104.351399) (end 172.311399 104.351399) (width 0.25) (layer F.Cu) (net 15))
   (segment (start 169.771399 104.351399) (end 170.96 105.54) (width 0.25) (layer B.Cu) (net 16) (status 20))
   (segment (start 137.43 103.067002) (end 138.719999 104.357001) (width 0.25) (layer B.Cu) (net 16) (status 10))

Commit message: updated package
Parts:
- U1: footprint Package_DIP:DIP-8_W7.62mm_SMDSocket_SmallPads -> Package_SO:SOIC-8_3.9x4.9mm_P1.27mm
- moved L1 5.38 mm to (131.8, 131.0)
- moved C3 3.06 mm to (144.4, 128.8)
- moved C2 2.66 mm to (144.4, 120.5)
- moved C1 0.62 mm to (151.0, 124.9)
Routing:
- net +3.3V: track 84.6 -> 80.9 mm
- net Net-(C2-Pad2): track 37.2 -> 33.7 mm
- net Net-(C2-Pad1): track 4.65 -> 2.45 mm
- net +24V: track 28.7 -> 30.2 mm
