File: Venta LW Controller.kicad_pcb (KiCad board)
At the start: 2 copper layers, 56 x 99.2 mm, 26 parts, among them J1 Conn_01x04, J2 Conn_02x05_Odd_Even, Q1 BSS138, Q2 BSS138, SW1 RST, SW2 FLASH, U1 LM2674N-3.3, U2 ESP32-WROOM-32

Commit message: updated parts
Parts:
- C1: value 22u -> 22uF; footprint Capacitor_Tantalum_SMD:CP_EIA-3216-18_Kemet-A -> Capacitor_Tantalum_SMD:CP_EIA-7343-31_Kemet-D
- C2: value 0.01u -> 0.01uF
- C3: value 100u -> 100uF
- C4: value 10n -> 10nF
- C5: value 47u -> 47uF
- L1: value 100u -> 100uH
- R2, R4, R5, R6, R7, R8: value 10k -> 10K
- moved D1 4.38 mm to (149.0, 119.6)
- moved J1 3.42 mm to (155.2, 116.0)
- moved C1 3.28 mm to (147.9, 126.0)
- moved C2 2.78 mm to (141.6, 120.5)
- moved C3 2.78 mm to (141.6, 128.8)
- moved U1 2.78 mm to (141.6, 124.1)
- moved SW2 2.04 mm to (159.5, 111.8)
- moved L1 0.64 mm to (131.2, 131.0)
Routing:
- net +3.3V: track 80.9 -> 90.3 mm
- net FLASH: track 50.6 -> 55.5 mm
- net TXD: track 52.7 -> 56.1 mm
- net RXD: track 55.4 -> 58.8 mm
- net Net-(C2-Pad2): track 33.7 -> 30.5 mm
- net +24V: track 30.2 -> 33.0 mm

Commit message: added and updated texts
Other:
- board text added: "3V3"
- board text added: "GND"
- board text added: "RXD"
- board text added: "TXD"
Changed lines of the file:
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@@
   (general
     (thickness 1.6)
-    (drawings 32)
+    (drawings 36)
     (tracks 173)
     (zones 0)
@@
     (tags resistor)
     (attr smd)
-    (fp_text reference R6 (at 4.0875 0 270) (layer F.SilkS)
+    (fp_text reference R6 (at 3.0875 0 270) (layer F.SilkS)
       (effects (font (size 1 1) (thickness 0.15)))
     )
@@
     (tags resistor)
     (attr smd)
-    (fp_text reference R5 (at 4.1 -0.102 270) (layer F.SilkS)
+    (fp_text reference R5 (at 3.1 -0.102 270) (layer F.SilkS)
       (effects (font (size 1 1) (thickness 0.15)))
     )
@@
     (tags resistor)
     (attr smd)
-    (fp_text reference R7 (at 4.1 0 270) (layer F.SilkS)
+    (fp_text reference R7 (at 3.1 0 270) (layer F.SilkS)
       (effects (font (size 1 1) (thickness 0.15)))
     )
@@
     (tags resistor)
     (attr smd)
-    (fp_text reference R4 (at 4.1 0 270) (layer F.SilkS)
+    (fp_text reference R4 (at 3.1 0 270) (layer F.SilkS)
       (effects (font (size 1 1) (thickness 0.15)))
     )
@@
     (tags resistor)
     (attr smd)
-    (fp_text reference R8 (at 4.1 0 270) (layer F.SilkS)
+    (fp_text reference R8 (at 3.1 0 270) (layer F.SilkS)
       (effects (font (size 1 1) (thickness 0.15)))
     )
@@
     )
   )
+  (gr_text GND (at 151.7142 116) (layer F.SilkS)
+    (effects (font (size 1 1) (thickness 0.15)))
+  )
+  (gr_text 3V3 (at 151.5618 113.45672) (layer F.SilkS)
+    (effects (font (size 1 1) (thickness 0.15)))
+  )
+  (gr_text RXD (at 151.57196 110.91672) (layer F.SilkS)
+    (effects (font (size 1 1) (thickness 0.15)))
+  )
+  (gr_text TXD (at 151.66848 108.37672) (layer F.SilkS)
+    (effects (font (size 1 1) (thickness 0.15)))
+  )
   (gr_text "ALITECS\nVenta LW Controller\nV2.0" (at 125.75 48.85) (layer F.SilkS)

Commit message: bumped version
Other:
- board text added: "ALITECS Venta LW Controller V2.1"
- board text removed: "ALITECS Venta LW Controller V2.0"
Changed lines of the file:
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@@
     (effects (font (size 1 1) (thickness 0.15)))
   )
-  (gr_text "ALITECS\nVenta LW Controller\nV2.0" (at 125.75 48.85) (layer F.SilkS)
+  (gr_text "ALITECS\nVenta LW Controller\nV2.1" (at 125.75 48.85) (layer F.SilkS)
     (effects (font (size 1 1) (thickness 0.15)) (justify left))
   )

Commit message: fixed transistor connection
Routing:
- net GPIO16: track 17.9 -> 19.8 mm
- net BTN_FANSPEED: track 42.2 -> 44.2 mm
Changed lines of the file:
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@@
     (thickness 1.6)
     (drawings 36)
-    (tracks 173)
+    (tracks 171)
     (zones 0)
     (modules 26)
@@
   (gr_line (start 148.5 52.76) (end 148.5 95.5) (layer Edge.Cuts) (width 0.05))
   (gr_arc (start 119 91) (end 127.499616 42.430432) (angle 25.3818742) (layer Edge.Cuts) (width 0.05))
-  (via (at 142.113 72.94372) (size 0.8) (drill 0.4) (layers F.Cu B.Cu) (net 1))
+  (via (at 142.748 72.94372) (size 0.8) (drill 0.4) (layers F.Cu B.Cu) (net 1))
   (via (at 130.08864 72.95388) (size 0.8) (drill 0.4) (layers F.Cu B.Cu) (net 1))
   (via (at 142.12824 92.49664) (size 0.8) (drill 0.4) (layers F.Cu B.Cu) (net 1))
@@
   (segment (start 139.39 97.5308) (end 139.39 95.7225) (width 0.25) (layer F.Cu) (net 13))
   (segment (start 173.4596 103) (end 170.0784 99.6188) (width 0.25) (layer F.Cu) (net 13))
-  (segment (start 133.934 102.632) (end 136.654011 105.352011) (width 0.25) (layer B.Cu) (net 15))
-  (segment (start 133.284 102.632) (end 133.934 102.632) (width 0.25) (layer B.Cu) (net 15) (status 10))
-  (segment (start 136.654011 105.352011) (end 161.457511 105.352011) (width 0.25) (layer B.Cu) (net 15))
   (segment (start 161.457511 105.352011) (end 161.457511 105.352011) (width 0.25) (layer B.Cu) (net 15))
   (via (at 161.457511 105.352011) (size 0.8) (drill 0.4) (layers F.Cu B.Cu) (net 15))
@@
   (segment (start 161.457511 105.352011) (end 162.458123 104.351399) (width 0.25) (layer F.Cu) (net 15))
   (segment (start 162.458123 104.351399) (end 172.311399 104.351399) (width 0.25) (layer F.Cu) (net 15))
+  (segment (start 133.984 102.682) (end 131.334 102.682) (width 0.25) (layer B.Cu) (net 15))
+  (segment (start 161.457511 105.352011) (end 136.654011 105.352011) (width 0.25) (layer B.Cu) (net 15))
+  (segment (start 136.654011 105.352011) (end 133.984 102.682) (width 0.25) (layer B.Cu) (net 15))
   (segment (start 169.771399 104.351399) (end 170.96 105.54) (width 0.25) (layer B.Cu) (net 16) (status 20))
   (segment (start 137.43 103.067002) (end 138.719999 104.357001) (width 0.25) (layer B.Cu) (net 16) (status 10))
@@
   (segment (start 140.145603 104.351399) (end 169.771399 104.351399) (width 0.25) (layer B.Cu) (net 16))
   (segment (start 140.140001 104.357001) (end 140.145603 104.351399) (width 0.25) (layer B.Cu) (net 16))
-  (via (at 139.4714 106.7308) (size 0.8) (drill 0.4) (layers F.Cu B.Cu) (net 17))
   (via (at 127.9144 97.5106) (size 0.8) (drill 0.4) (layers F.Cu B.Cu) (net 17))
-  (segment (start 139.4714 106.7308) (end 137.1346 106.7308) (width 0.25) (layer F.Cu) (net 17))
-  (segment (start 137.1346 106.7308) (end 127.9144 97.5106) (width 0.25) (layer F.Cu) (net 17))
   (segment (start 127.9144 89.4678) (end 127.9234 89.4588) (width 0.25) (layer B.Cu) (net 17))
   (segment (start 127.9144 97.5106) (end 127.9144 89.4678) (width 0.25) (layer B.Cu) (net 17))
@@
   (segment (start 163.9552 111.77) (end 165.99152 111.77) (width 0.25) (layer B.Cu) (net 17))
   (segment (start 165.99676 111.77524) (end 159.49676 111.77524) (width 0.25) (layer B.Cu) (net 17))
-  (segment (start 154.26436 106.7308) (end 139.4714 106.7308) (width 0.25) (layer B.Cu) (net 17))
-  (segment (start 156.80944 106.7308) (end 154.26436 106.7308) (width 0.25) (layer B.Cu) (net 17))
-  (segment (start 157.48508 107.40644) (end 156.80944 106.7308) (width 0.25) (layer B.Cu) (net 17))
-  (segment (start 159.49676 111.77524) (end 157.48508 109.76356) (width 0.25) (layer B.Cu) (net 17))
-  (segment (start 157.48508 109.76356) (end 157.48508 107.40644) (width 0.25) (layer B.Cu) (net 17))
-  (segment (start 129.369389 87.114789) (end 129.1734 86.9188) (width 0.25) (layer B.Cu) (net 32))
-  (segment (start 129.1734 86.9188) (end 127.9234 86.9188) (width 0.25) (layer B.Cu) (net 32))
-  (segment (start 129.369389 97.2078) (end 129.369389 87.114789) (width 0.25) (layer B.Cu) (net 32))
-  (segment (start 131.384 99.222411) (end 129.369389 97.2078) (width 0.25) (layer B.Cu) (net 32))
-  (segment (start 131.384 102.632) (end 131.384 99.222411) (width 0.25) (layer B.Cu) (net 32))
+  (via (at 136.8933 106.4895) (size 0.8) (drill 0.4) (layers F.Cu B.Cu) (net 17))
+  (segment (start 127.9144 97.5106) (end 136.8933 106.4895) (width 0.25) (layer F.Cu) (net 17))
+  (segment (start 137.458985 106.4895) (end 136.8933 106.4895) (width 0.25) (layer B.Cu) (net 17))
+  (segment (start 157.0609 106.4895) (end 137.458985 106.4895) (width 0.25) (layer B.Cu) (net 17))
+  (segment (start 159.49676 111.77524) (end 159.49676 108.92536) (width 0.25) (layer B.Cu) (net 17))
+  (segment (start 159.49676 108.92536) (end 157.0609 106.4895) (width 0.25) (layer B.Cu) (net 17))
+  (segment (start 131.334 104.532) (end 131.334 104.582) (width 0.25) (layer B.Cu) (net 32))
+  (segment (start 129.369389 102.567389) (end 131.334 104.532) (width 0.25) (layer B.Cu) (net 32))
+  (segment (start 129.369389 87.114789) (end 129.369389 102.567389) (width 0.25) (layer B.Cu) (net 32))
+  (segment (start 127.9234 86.9188) (end 129.1734 86.9188) (width 0.25) (layer B.Cu) (net 32))
+  (segment (start 129.1734 86.9188) (end 129.369389 87.114789) (width 0.25) (layer B.Cu) (net 32))
   (segment (start 129.1734 85.6488) (end 127.9234 85.6488) (width 0.25) (layer B.Cu) (net 45))
   (segment (start 129.8194 86.2948) (end 129.1734 85.6488) (width 0.25) (layer B.Cu) (net 45))

Commit message: cleaned circuits
Routing:
- net RST: track 81.7 -> 79.3 mm
- net FLASH: track 55.8 -> 53.7 mm
Changed lines of the file:
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@@
     (thickness 1.6)
     (drawings 36)
-    (tracks 171)
+    (tracks 169)
     (zones 0)
     (modules 26)
@@
   (segment (start 174.720987 111.77) (end 169.6352 111.77) (width 0.25) (layer B.Cu) (net 6))
   (segment (start 176.1352 111.77) (end 174.720987 111.77) (width 0.25) (layer B.Cu) (net 6))
+  (segment (start 146.932599 95.472199) (end 146.5326 95.0722) (width 0.25) (layer B.Cu) (net 6))
   (segment (start 149.810409 98.350009) (end 146.932599 95.472199) (width 0.25) (layer B.Cu) (net 6))
-  (segment (start 146.932599 95.472199) (end 146.5326 95.0722) (width 0.25) (layer B.Cu) (net 6))
-  (segment (start 177.6476 100.16744) (end 175.830169 98.350009) (width 0.25) (layer B.Cu) (net 6))
-  (segment (start 175.830169 98.350009) (end 149.810409 98.350009) (width 0.25) (layer B.Cu) (net 6))
-  (segment (start 176.1352 111.77) (end 177.6476 110.2576) (width 0.25) (layer B.Cu) (net 6))
-  (segment (start 177.6476 110.2576) (end 177.6476 100.16744) (width 0.25) (layer B.Cu) (net 6))
+  (segment (start 173.864209 98.350009) (end 149.810409 98.350009) (width 0.25) (layer B.Cu) (net 6))
+  (segment (start 176.149 100.6348) (end 173.864209 98.350009) (width 0.25) (layer B.Cu) (net 6))
+  (segment (start 176.1352 111.77) (end 176.149 111.7562) (width 0.25) (layer B.Cu) (net 6))
+  (segment (start 176.149 111.7562) (end 176.149 100.6348) (width 0.25) (layer B.Cu) (net 6))
   (via (at 136.906 108.3056) (size 0.8) (drill 0.4) (layers F.Cu B.Cu) (net 7))
   (via (at 126.11608 76.758804) (size 0.8) (drill 0.4) (layers F.Cu B.Cu) (net 7))
@@
   (segment (start 127.9144 89.4678) (end 127.9234 89.4588) (width 0.25) (layer B.Cu) (net 17))
   (segment (start 127.9144 97.5106) (end 127.9144 89.4678) (width 0.25) (layer B.Cu) (net 17))
-  (segment (start 165.99152 111.77) (end 165.99676 111.77524) (width 0.25) (layer B.Cu) (net 17))
-  (segment (start 163.9552 111.77) (end 165.99152 111.77) (width 0.25) (layer B.Cu) (net 17))
-  (segment (start 165.99676 111.77524) (end 159.49676 111.77524) (width 0.25) (layer B.Cu) (net 17))
   (via (at 136.8933 106.4895) (size 0.8) (drill 0.4) (layers F.Cu B.Cu) (net 17))
   (segment (start 127.9144 97.5106) (end 136.8933 106.4895) (width 0.25) (layer F.Cu) (net 17))
@@
   (segment (start 159.49676 111.77524) (end 159.49676 108.92536) (width 0.25) (layer B.Cu) (net 17))
   (segment (start 159.49676 108.92536) (end 157.0609 106.4895) (width 0.25) (layer B.Cu) (net 17))
+  (segment (start 159.49676 111.77524) (end 165.99676 111.77524) (width 0.25) (layer B.Cu) (net 17))
   (segment (start 131.334 104.532) (end 131.334 104.582) (width 0.25) (layer B.Cu) (net 32))
   (segment (start 129.369389 102.567389) (end 131.334 104.532) (width 0.25) (layer B.Cu) (net 32))
